File: schematic/fautonling-schematic.sch (KiCad schematic (older format))
At the start: 16 parts, among them M1 AVC BA10033B12U, M2 AVC BA10033B12U, Q1 IRFZ44N, U1 L78L05_TO92, U2 ATtiny13A-SU, U3 LM35-LP

Commit message: Finish off schematic
The fans finally arrived, testing ensued, this is t'result
Parts:
- removed M1, M2: AVC BA10033B12U, symbol Motor:Fan
- added D2, D3: 1N5819, symbol Device:D_Schottky
- added M1, M2: AVC BA10033B12U, symbol Motor:Fan_3pin
- renumbered D2 to D4
Connections:
- wire segments 36 -> 43
Other:
- note removed: "3-pin connector: if tacho -> steal one LED pin for that"
- note removed: "rgb pins?"
- moved on the sheet: Q1

Commit message: Transistors are Good, actually
Parts:
- added Q2: BC337, Package_TO_SOT_THT:TO-92_Inline, symbol Transistor_BJT:BC337
- added R1: 2200R, symbol Device:R
- added R2: 4700R, symbol Device:R
Connections:
- wire segments 43 -> 45
Other:
- note added: "Does this puny "snubber network" for 3A total of fan?"
Changed lines of the file:
@@
 NoConn ~ 2800 4000
-$Comp
-L power:+5V #PWR?
-U 1 1 5BF5CCE4
-P 9000 850
-F 0 "#PWR?" H 9000 700 50  0001 C CNN
-F 1 "+5V" V 9015 978 50  0000 L CNN
-F 2 "" H 9000 850 50  0001 C CNN
-F 3 "" H 9000 850 50  0001 C CNN
-	1    9000 850
-	1    0    0    -1
-$EndComp
 $Comp
 L Device:R_Variable R1
@@
 U 1 1 5BF5E604
 P 4350 3000
-F 0 "Q1" H 4578 3046 50  0000 L CNN
-F 1 "IRFZ44N" H 4578 2955 50  0000 L CNN
+F 0 "Q1" H 4555 3046 50  0000 L CNN
+F 1 "IRFZ44N" H 4555 2955 50  0000 L CNN
 F 2 "Package_TO_SOT_THT:TO-220-3_Vertical" H 4600 2925 50  0001 L CIN
 F 3 "" H 4350 3000 50  0001 L CNN
@@
 	3950 2500 3950 1850
 Wire Wire Line
-	2800 3600 9800 3600
-Wire Wire Line
-	9800 1700 9800 3600
+	2800 3600 9150 3600
 Wire Wire Line
 	9000 1700 9000 2000
@@
 	0    -1   -1   0
 $EndComp
+Text Notes 6050 3050 0    50   ~ 0
+Does this puny "snubber network" for 3A total of fan?
+$Comp
+L power:+12V #PWR?
+U 1 1 5C011846
+P 9000 850
+F 0 "#PWR?" H 9000 700 50  0001 C CNN
+F 1 "+12V" V 9015 978 50  0000 L CNN
+F 2 "" H 9000 850 50  0001 C CNN
+F 3 "" H 9000 850 50  0001 C CNN
+	1    9000 850
+	1    0    0    -1
+$EndComp
+$Comp
+L Transistor_BJT:BC337 Q2
+U 1 1 5C012DF0
+P 9700 3900
+F 0 "Q2" H 9891 3946 50  0000 L CNN
+F 1 "BC337" H 9891 3855 50  0000 L CNN
+F 2 "Package_TO_SOT_THT:TO-92_Inline" H 9900 3825 50  0001 L CIN
+F 3 "http://www.nxp.com/documents/data_sheet/BC817_BC817W_BC337.pdf" H 9700 3900 50  0001 L CNN
+	1    9700 3900
+	1    0    0    -1
+$EndComp
+$Comp
+L Device:R R1
+U 1 1 5C014109
+P 9150 3750
+F 0 "R1" H 9220 3796 50  0000 L CNN
+F 1 "2200R" H 9220 3705 50  0000 L CNN
+F 2 "" V 9080 3750 50  0001 C CNN
+F 3 "~" H 9150 3750 50  0001 C CNN
+	1    9150 3750
+	1    0    0    -1
+$EndComp
+$Comp
+L Device:R R2
+U 1 1 5C0144C7
+P 9150 4050
+F 0 "R2" H 9220 4096 50  0000 L CNN
+F 1 "4700R" H 9220 4005 50  0000 L CNN
+F 2 "" V 9080 4050 50  0001 C CNN
+F 3 "~" H 9150 4050 50  0001 C CNN
+	1    9150 4050
+	1    0    0    -1
+$EndComp
+Wire Wire Line
+	9150 3900 9500 3900
+Connection ~ 9150 3900
+Wire Wire Line
+	9800 1700 9800 3700
+$Comp
+L power:GND #PWR?
+U 1 1 5C018A27
+P 9150 4200
+F 0 "#PWR?" H 9150 3950 50  0001 C CNN
+F 1 "GND" H 9155 4027 50  0000 C CNN
+F 2 "" H 9150 4200 50  0001 C CNN
+F 3 "" H 9150 4200 50  0001 C CNN
+	1    9150 4200
+	1    0    0    -1
+$EndComp
+$Comp
+L power:GND #PWR?
+U 1 1 5C01918C
+P 9800 4200
+F 0 "#PWR?" H 9800 3950 50  0001 C CNN
+F 1 "GND" H 9805 4027 50  0000 C CNN
+F 2 "" H 9800 4200 50  0001 C CNN
+F 3 "" H 9800 4200 50  0001 C CNN
+	1    9800 4200
+	1    0    0    -1
+$EndComp
+Wire Wire Line
+	9800 4100 9800 4200
 $EndSCHEMATC

Commit message: Add datasheets and footprints to all elements except the potentiometers (I've no idea which footprint matches mine?)
Parts:
- C1, C2, C3, C5: footprint (none) -> Capacitor_THT:C_Rect_L7.0mm_W2.5mm_P5.00mm
- C4: footprint (none) -> Capacitor_THT:CP_Radial_Tantal_D4.5mm_P2.50mm
- D1: footprint (none) -> LED_THT:LED_D5.0mm-4
- D2, D3, D4: footprint (none) -> Diode_THT:D_DO-41_SOD81_P7.62mm_Horizontal
- R4: renamed from R1; footprint (none) -> Resistor_THT:R_Axial_DIN0204_L3.6mm_D1.6mm_P7.62mm_Horizontal
- R5: renamed from R2; footprint (none) -> Resistor_THT:R_Axial_DIN0204_L3.6mm_D1.6mm_P7.62mm_Horizontal
- U2: footprint Package_SO:SOIJ-8_5.3x5.3mm_P1.27mm -> Package_DIP:DIP-8_W7.62mm_Socket
- U3: footprint (none) -> Package_TO_SOT_THT:TO-92_Inline
Changed lines of the file:
@@
 F 0 "U2" H 1670 3846 50  0000 R CNN
 F 1 "ATtiny13A-SU" H 1670 3755 50  0000 R CNN
-F 2 "Package_SO:SOIJ-8_5.3x5.3mm_P1.27mm" H 2200 3800 50  0001 C CIN
+F 2 "Package_DIP:DIP-8_W7.62mm_Socket" H 2200 3800 50  0001 C CIN
 F 3 "http://ww1.microchip.com/downloads/en/DeviceDoc/doc8126.pdf" H 2200 3800 50  0001 C CNN
 	1    2200 3800
@@
 F 0 "C1" H 1285 1704 50  0000 R CNN
 F 1 "370-470nF" H 1285 1795 50  0000 R CNN
-F 2 "" H 1438 1600 50  0001 C CNN
+F 2 "Capacitor_THT:C_Rect_L7.0mm_W2.5mm_P5.00mm" H 1438 1600 50  0001 C CNN
 F 3 "~" H 1400 1750 50  0001 C CNN
 	1    1400 1750
@@
 F 0 "C4" H 2615 1796 50  0000 L CNN
 F 1 "33μF" H 2615 1705 50  0000 L CNN
-F 2 "" H 2538 1600 50  0001 C CNN
+F 2 "Capacitor_THT:CP_Radial_Tantal_D4.5mm_P2.50mm" H 2538 1600 50  0001 C CNN
 F 3 "~" H 2500 1750 50  0001 C CNN
 	1    2500 1750
@@
 F 0 "D1" H 9000 1547 50  0000 C CNN
 F 1 "LED_RABG" H 9000 1456 50  0000 C CNN
-F 2 "" H 9000 1000 50  0001 C CNN
+F 2 "LED_THT:LED_D5.0mm-4" H 9000 1000 50  0001 C CNN
 F 3 "~" H 9000 1000 50  0001 C CNN
 	1    9000 1050
@@
 F 0 "C2" V 2052 3050 50  0000 C CNN
 F 1 "100nF" V 1961 3050 50  0000 C CNN
-F 2 "" H 1838 2900 50  0001 C CNN
+F 2 "Capacitor_THT:C_Rect_L7.0mm_W2.5mm_P5.00mm" H 1838 2900 50  0001 C CNN
 F 3 "~" H 1800 3050 50  0001 C CNN
 	1    1800 3050
@@
 F 1 "IRFZ44N" H 4555 2955 50  0000 L CNN
 F 2 "Package_TO_SOT_THT:TO-220-3_Vertical" H 4600 2925 50  0001 L CIN
-F 3 "" H 4350 3000 50  0001 L CNN
+F 3 "https://www.mouser.com/catalog/specsheets/irfz44n.pdf" H 4350 3000 50  0001 L CNN
 	1    4350 3000
 	1    0    0    -1
@@
 F 0 "U3" H 1870 5946 50  0000 R CNN
 F 1 "LM35-LP" H 1870 5855 50  0000 R CNN
-F 2 "" H 2250 5650 50  0001 L CNN
+F 2 "Package_TO_SOT_THT:TO-92_Inline" H 2250 5650 50  0001 L CNN
 F 3 "http://www.ti.com/lit/ds/symlink/lm35.pdf" H 2200 5900 50  0001 C CNN
 	1    2200 5900
@@
 F 0 "C3" V 2052 5450 50  0000 C CNN
 F 1 "100nF" V 1961 5450 50  0000 C CNN
-F 2 "" H 1838 5300 50  0001 C CNN
+F 2 "Capacitor_THT:C_Rect_L7.0mm_W2.5mm_P5.00mm" H 1838 5300 50  0001 C CNN
 F 3 "~" H 1800 5450 50  0001 C CNN
 	1    1800 5450
@@
 F 0 "D2" H 7800 2066 50  0000 C CNN
 F 1 "1N5819" H 7800 1975 50  0000 C CNN
-F 2 "" H 7800 1850 50  0001 C CNN
-F 3 "~" H 7800 1850 50  0001 C CNN
+F 2 "Diode_THT:D_DO-41_SOD81_P7.62mm_Horizontal" H 7800 1850 50  0001 C CNN
+F 3 "https://www.diodes.com/assets/Datasheets/ds23001.pdf" H 7800 1850 50  0001 C CNN
 	1    7800 1850
 	1    0    0    -1
@@
 F 0 "D3" H 8600 2216 50  0000 C CNN
 F 1 "1N5819" H 8600 2125 50  0000 C CNN
-F 2 "" H 8600 2000 50  0001 C CNN
-F 3 "~" H 8600 2000 50  0001 C CNN
+F 2 "Diode_THT:D_DO-41_SOD81_P7.62mm_Horizontal" H 8600 2000 50  0001 C CNN
+F 3 "https://www.diodes.com/assets/Datasheets/ds23001.pdf" H 8600 2000 50  0001 C CNN
 	1    8600 2000
 	1    0    0    -1
@@
 F 0 "C5" H 6765 2596 50  0000 L CNN
 F 1 "100nF" H 6765 2505 50  0000 L CNN
-F 2 "" H 6688 2400 50  0001 C CNN
+F 2 "Capacitor_THT:C_Rect_L7.0mm_W2.5mm_P5.00mm" H 6688 2400 50  0001 C CNN
 F 3 "~" H 6650 2550 50  0001 C CNN
 	1    6650 2550
@@
 F 0 "D4" V 7146 2471 50  0000 R CNN
 F 1 "1N5819" V 7055 2471 50  0000 R CNN
-F 2 "" H 7100 2550 50  0001 C CNN
-F 3 "~" H 7100 2550 50  0001 C CNN
+F 2 "Diode_THT:D_DO-41_SOD81_P7.62mm_Horizontal" H 7100 2550 50  0001 C CNN
+F 3 "https://www.diodes.com/assets/Datasheets/ds23001.pdf" H 7100 2550 50  0001 C CNN
 	1    7100 2550
 	0    -1   -1   0
@@
 $EndComp
 $Comp
-L Device:R R1
+L Device:R R4
 U 1 1 5C014109
 P 9150 3750
-F 0 "R1" H 9220 3796 50  0000 L CNN
+F 0 "R4" H 9220 3796 50  0000 L CNN
 F 1 "2200R" H 9220 3705 50  0000 L CNN
-F 2 "" V 9080 3750 50  0001 C CNN
+F 2 "Resistor_THT:R_Axial_DIN0204_L3.6mm_D1.6mm_P7.62mm_Horizontal" V 9080 3750 50  0001 C CNN
 F 3 "~" H 9150 3750 50  0001 C CNN
 	1    9150 3750
@@
 $EndComp
 $Comp
-L Device:R R2
+L Device:R R5
 U 1 1 5C0144C7
 P 9150 4050
-F 0 "R2" H 9220 4096 50  0000 L CNN
+F 0 "R5" H 9220 4096 50  0000 L CNN
 F 1 "4700R" H 9220 4005 50  0000 L CNN
-F 2 "" V 9080 4050 50  0001 C CNN
+F 2 "Resistor_THT:R_Axial_DIN0204_L3.6mm_D1.6mm_P7.62mm_Horizontal" V 9080 4050 50  0001 C CNN
 F 3 "~" H 9150 4050 50  0001 C CNN
 	1    9150 4050

Commit message: But actually tho
Parts:
- removed C1: 370-470nF, Capacitor_THT:C_Rect_L7.0mm_W2.5mm_P5.00mm, symbol Device:C
- removed C3: 100nF, Capacitor_THT:C_Rect_L7.0mm_W2.5mm_P5.00mm, symbol Device:C
- removed C4: 33μF, Capacitor_THT:CP_Radial_Tantal_D4.5mm_P2.50mm, symbol Device:C
- removed D1: LED_RABG, LED_THT:LED_D5.0mm-4, symbol Device:LED_RABG
- removed D2, D3, D4: 1N5819, Diode_THT:D_DO-41_SOD81_P7.62mm_Horizontal, symbol Device:D_Schottky
- removed Q2: BC337, Package_TO_SOT_THT:TO-92_Inline, symbol Transistor_BJT:BC337
- removed R1, R2, R3: 5000R, symbol Device:R_Variable
- removed R4: 2200R, Resistor_THT:R_Axial_DIN0204_L3.6mm_D1.6mm_P7.62mm_Horizontal, symbol Device:R
- removed R5: 4700R, Resistor_THT:R_Axial_DIN0204_L3.6mm_D1.6mm_P7.62mm_Horizontal, symbol Device:R
- removed U1: L78L05_TO92, Package_TO_SOT_THT:TO-92_Inline, symbol Regulator_Linear:L78L05_TO92
- removed U2: ATtiny13A-SU, Package_DIP:DIP-8_W7.62mm_Socket, symbol MCU_Microchip_ATtiny:ATtiny13A-SU
- removed U3: LM35-LP, Package_TO_SOT_THT:TO-92_Inline, symbol Sensor_Temperature:LM35-LP
- added D1: 1N4007, symbol Device:D
- added D2: LED, symbol Device:LED
- added R1, R2: 4700R, symbol Device:R
- added RV1: 5000RTRIM, symbol Device:R_POT_TRIM
- added U1: LM335Z, symbol Device:LM335Z
- added U2: LM339, symbol Comparator:LM339
- renumbered C5 to C1
Connections:
- net labels removed: +5V
- wire segments 45 -> 20
Other:
- note removed: "Close to body"
- note removed: "Does this puny "snubber network" for 3A total of fan?"
